File: barometer.sch (EAGLE design)
At the start: 105 parts, among them IC1 TPS5410, IC2 ZPA2326-0311A-R, IC3 MIC5225-3.3v, Q1 BC817, U1 LTC2850, U2 PCA9306, U3 DAC8574, U4 XTR117, U5 XC6215XC6215B182NR, U6 MAX3221, U7 Tiny85-20-SMT, X1 1751248, X2 1751264

Commit message: Remove trace in solder jumper SJ3
Parts:
- SJ3: value SOLDERJUMPERTRACE -> SOLDERJUMPERNO; device SparkFun-Retired-0:SOLDERJUMPERTRACE -> SparkFun-Retired-0:SOLDERJUMPERNO
Changed lines of the file:
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@@
 <part name="TP13" library="testpad" library_urn="urn:adsk.eagle:library:385" deviceset="PTR1" device="B1,27" package3d_urn="urn:adsk.eagle:package:27944/1"/>
 <part name="U7" library="SparkFun-Retired-0" deviceset="ATTINY45" device="TINY85-20-SMT" value="Tiny85-20-SMT"/>
-<part name="SJ3" library="SparkFun-Retired-0" deviceset="SOLDERJUMPER" device="TRACE"/>
 <part name="SJ9" library="SparkFun-Retired-0" deviceset="SOLDERJUMPER" device="TRACE"/>
 <part name="SJ8" library="SparkFun-Retired-0" deviceset="SOLDERJUMPER" device="TRACE"/>
@@
 <part name="TP19" library="testpad" library_urn="urn:adsk.eagle:library:385" deviceset="PTR1" device="B1,27" package3d_urn="urn:adsk.eagle:package:27944/1"/>
 <part name="JP3" library="microbuilder" deviceset="HEADER-1X3" device="SMT" value="Analog Output Format 2"/>
+<part name="SJ3" library="SparkFun-Retired-0" deviceset="SOLDERJUMPER" device="NO"/>
 </parts>
 <sheets>
@@
 <attribute name="NAME" x="223.52" y="147.32" size="1.778" layer="95" font="vector" rot="MR0"/>
 </instance>
+<instance part="SJ9" gate="1" x="41.91" y="134.62" smashed="yes" rot="R90">
+<attribute name="NAME" x="39.37" y="132.08" size="1.778" layer="95" font="vector" rot="R90"/>
+</instance>
+<instance part="SJ8" gate="1" x="49.53" y="134.62" smashed="yes" rot="R90">
+<attribute name="NAME" x="46.99" y="132.08" size="1.778" layer="95" font="vector" rot="R90"/>
+</instance>
+<instance part="SJ11" gate="1" x="57.15" y="134.62" smashed="yes" rot="R90">
+<attribute name="NAME" x="54.61" y="132.08" size="1.778" layer="95" font="vector" rot="R90"/>
+</instance>
+<instance part="SJ10" gate="1" x="64.77" y="134.62" smashed="yes" rot="R90">
+<attribute name="NAME" x="62.23" y="132.08" size="1.778" layer="95" font="vector" rot="R90"/>
+</instance>
+<instance part="SJ12" gate="1" x="72.39" y="134.62" smashed="yes" rot="R90">
+<attribute name="NAME" x="69.85" y="132.08" size="1.778" layer="95" font="vector" rot="R90"/>
+</instance>
+<instance part="SJ1" gate="1" x="80.01" y="134.62" smashed="yes" rot="R90">
+<attribute name="NAME" x="77.47" y="132.08" size="1.778" layer="95" font="vector" rot="R90"/>
+</instance>
+<instance part="SJ2" gate="1" x="87.63" y="134.62" smashed="yes" rot="R90">
+<attribute name="NAME" x="85.09" y="132.08" size="1.778" layer="95" font="vector" rot="R90"/>
+</instance>
+<instance part="PAD5" gate="1" x="48.26" y="43.18" smashed="yes">
+<attribute name="VALUE" x="47.117" y="39.878" size="1.778" layer="96"/>
+</instance>
+<instance part="PAD3" gate="1" x="48.26" y="45.72" smashed="yes">
+<attribute name="VALUE" x="47.117" y="42.418" size="1.778" layer="96"/>
+</instance>
+<instance part="PAD1" gate="1" x="48.26" y="48.26" smashed="yes">
+<attribute name="VALUE" x="47.117" y="44.958" size="1.778" layer="96"/>
+</instance>
+<instance part="PAD2" gate="1" x="45.72" y="48.26" smashed="yes" rot="R180">
+<attribute name="VALUE" x="46.863" y="51.562" size="1.778" layer="96" rot="R180"/>
+</instance>
+<instance part="PAD4" gate="1" x="45.72" y="45.72" smashed="yes" rot="R180">
+<attribute name="VALUE" x="46.863" y="49.022" size="1.778" layer="96" rot="R180"/>
+</instance>
+<instance part="PAD6" gate="1" x="45.72" y="43.18" smashed="yes" rot="R180">
+<attribute name="VALUE" x="46.863" y="46.482" size="1.778" layer="96" rot="R180"/>
+</instance>
 <instance part="SJ3" gate="1" x="34.29" y="134.62" smashed="yes" rot="R90">
 <attribute name="NAME" x="31.75" y="132.08" size="1.778" layer="95" font="vector" rot="R90"/>
-</instance>
-<instance part="SJ9" gate="1" x="41.91" y="134.62" smashed="yes" rot="R90">
-<attribute name="NAME" x="39.37" y="132.08" size="1.778" layer="95" font="vector" rot="R90"/>
-</instance>
-<instance part="SJ8" gate="1" x="49.53" y="134.62" smashed="yes" rot="R90">
-<attribute name="NAME" x="46.99" y="132.08" size="1.778" layer="95" font="vector" rot="R90"/>
-</instance>
-<instance part="SJ11" gate="1" x="57.15" y="134.62" smashed="yes" rot="R90">
-<attribute name="NAME" x="54.61" y="132.08" size="1.778" layer="95" font="vector" rot="R90"/>
-</instance>
-<instance part="SJ10" gate="1" x="64.77" y="134.62" smashed="yes" rot="R90">
-<attribute name="NAME" x="62.23" y="132.08" size="1.778" layer="95" font="vector" rot="R90"/>
-</instance>
-<instance part="SJ12" gate="1" x="72.39" y="134.62" smashed="yes" rot="R90">
-<attribute name="NAME" x="69.85" y="132.08" size="1.778" layer="95" font="vector" rot="R90"/>
-</instance>
-<instance part="SJ1" gate="1" x="80.01" y="134.62" smashed="yes" rot="R90">
-<attribute name="NAME" x="77.47" y="132.08" size="1.778" layer="95" font="vector" rot="R90"/>
-</instance>
-<instance part="SJ2" gate="1" x="87.63" y="134.62" smashed="yes" rot="R90">
-<attribute name="NAME" x="85.09" y="132.08" size="1.778" layer="95" font="vector" rot="R90"/>
-</instance>
-<instance part="PAD5" gate="1" x="48.26" y="43.18" smashed="yes">
-<attribute name="VALUE" x="47.117" y="39.878" size="1.778" layer="96"/>
-</instance>
-<instance part="PAD3" gate="1" x="48.26" y="45.72" smashed="yes">
-<attribute name="VALUE" x="47.117" y="42.418" size="1.778" layer="96"/>
-</instance>
-<instance part="PAD1" gate="1" x="48.26" y="48.26" smashed="yes">
-<attribute name="VALUE" x="47.117" y="44.958" size="1.778" layer="96"/>
-</instance>
-<instance part="PAD2" gate="1" x="45.72" y="48.26" smashed="yes" rot="R180">
-<attribute name="VALUE" x="46.863" y="51.562" size="1.778" layer="96" rot="R180"/>
-</instance>
-<instance part="PAD4" gate="1" x="45.72" y="45.72" smashed="yes" rot="R180">
-<attribute name="VALUE" x="46.863" y="49.022" size="1.778" layer="96" rot="R180"/>
-</instance>
-<instance part="PAD6" gate="1" x="45.72" y="43.18" smashed="yes" rot="R180">
-<attribute name="VALUE" x="46.863" y="46.482" size="1.778" layer="96" rot="R180"/>
 </instance>
 </instances>
@@
 <net name="SDA_3V3" class="0">
 <segment>
-<pinref part="SJ3" gate="1" pin="2"/>
 <wire x1="34.29" y1="139.7" x2="34.29" y2="142.24" width="0.1524" layer="91"/>
 <label x="35.56" y="143.51" size="1.778" layer="95" font="vector" rot="R90"/>
+<pinref part="SJ3" gate="1" pin="2"/>
 </segment>
 </net>
@@
 <net name="B0" class="0">
 <segment>
-<pinref part="SJ3" gate="1" pin="1"/>
 <wire x1="34.29" y1="127" x2="34.29" y2="129.54" width="0.1524" layer="91"/>
 <label x="33.02" y="125.73" size="1.778" layer="95" font="vector" rot="R270"/>
-</segment>
-<segment>
+<pinref part="SJ3" gate="1" pin="1"/>
+</segment>
+<segment>
